File: eagle/mojoafe/mojoafe.brd (EAGLE design)
At the start: 68.2 x 55.9 mm, 37 parts, among them IC1 MAX9939, IC2 MAX9939, IC3 MAX9939, IC4 MAX11044B, IC5 MAX9939, J1 SMB50R, J2 SMB50R, J3 SMB50R, J4 SMB50R

Commit message: finished mojo afe PCB, generated CAM files and BoM
Parts:
- added C23, C24: 1u, resistor:C0603K
- added IC10, IC9: TLV70033, custom:SOT5
- added IC6, IC7, IC8: ADS8327, custom:TSSOP16
- added R5, R6, R7, R8: 20R, resistor:R0603
- added TP1, TP2, TP3, TP4, TP5, TP6, TP7, TP8, TP9: (no value), pinhead:1X01
- C1, C10, C12, C3, C4, C9: value .1u -> 10u
- C11, C2: value .1u -> 470p
- C13, C14: value .1u -> 1u
- C5, C8: value 22u -> 470p; device resistor:C0805K -> resistor:C0603K
- C6, C7: value 22u -> 10u; device resistor:C0805K -> resistor:C0603K
- IC4: value MAX11044B -> ADS8327; device custom:TQFP64 -> custom:TSSOP16
- JP1, JP2: device pinhead:2X25 -> pinhead:2X20
- R1, R2, R3, R4: value 100R -> 20R
- moved C18 86.0 mm to (16.4, 35.9), turned to 180 degrees
- moved C16 86.0 mm to (16.1, 44.3), turned to 180 degrees
- moved C20 85.5 mm to (16.4, 27.1), turned to 180 degrees
- moved C22 85.0 mm to (16.4, 18.2), turned to 180 degrees
- moved C17 80.6 mm to (16.4, 34.5), turned to 180 degrees
- moved C15 80.5 mm to (16.1, 42.9), turned to 180 degrees
- moved C19 80.1 mm to (16.4, 25.7), turned to 180 degrees
- moved C21 79.6 mm to (16.4, 16.8), turned to 180 degrees
- moved C6 65.6 mm to (32.9, 34.0), turned to 180 degrees
- moved C7 59.2 mm to (28.8, 25.1)
- moved C8 58.2 mm to (25.9, 21.6), turned to 270 degrees
- moved C5 55.9 mm to (25.9, 30.5), turned to 270 degrees
- moved C14 38.3 mm to (9.02, 47.8), turned to 180 degrees
- moved C13 32.3 mm to (16.1, 46.1), turned to 0 degrees
- moved C2 26.4 mm to (25.9, 39.4), turned to 270 degrees
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Connections:
- removed net !CS: IC4.62, JP1.36
- removed net !EOC: IC4.18, JP1.18
- removed net !RD: IC4.63, JP1.35
- removed net !WR: IC4.61, JP1.37
- removed net +5V: C10.1, C11.1, C12.1, C13.1, C14.1, C15.1, C16.1, C17.1, C18.1, C19.1, C20.1, C21.1, C22.1, C9.1, IC1.9, IC2.9, IC3.9, IC4.24, IC4.29, IC4.35, IC4.46, IC4.52, IC4.57, IC5.9
- removed net CONVST: IC4.19, JP1.17
- removed net DB0: IC4.17, JP1.19
- removed net DB1: IC4.16, JP1.20
- removed net DB10: IC4.5, JP1.29
- removed net DB11: IC4.4, JP1.30
- removed net DB12: IC4.3, JP1.31
- removed net DB13: IC4.2, JP1.32
- removed net DB14: IC4.1, JP1.33
- removed net DB15: IC4.64, JP1.34
- removed net DB2: IC4.15, JP1.21
- removed net DB3: IC4.14, JP1.22
- removed net DB4: IC4.13, JP1.23
- removed net DB5: IC4.12, JP1.24
- removed net DB6: IC4.11, JP1.25
- removed net DB7: IC4.10, JP1.26
- removed net DB8: IC4.7, JP1.27
- removed net DB9: IC4.6, JP1.28
- removed net N$11: IC5.8, R4.1
- removed net REFIO: C1.1, IC4.41
- removed net SHDN: IC4.20, JP1.16
- new net !CONVST1: IC6.9, JP1.32
- new net !CONVST2: IC4.9, JP1.38
- new net !CONVST3: IC7.9, JP2.34
- new net !CONVST4: IC8.9, JP2.28
- new net !CS1: IC6.11, JP1.30
- new net !CS2: IC4.11, JP1.36
- new net !CS3: IC7.11, JP2.36
- new net !CS4: IC8.11, JP2.30
- new net +3V3A: C1.1, C10.1, C13.1, C15.1, C16.1, C17.1, C18.1, C19.1, C20.1, C21.1, C22.1, C4.1, C7.1, IC1.9, IC2.9, IC3.9, IC4.1, IC4.7, IC5.9, IC6.1, IC6.7, IC7.1, IC7.7, IC8.1, IC8.7, IC9.5
- new net +3V3D: C12.1, C23.1, C3.1, C6.1, C9.1, IC10.5, IC4.16, IC6.16, IC7.16, IC8.16
- new net EOC1: IC6.10, JP1.31
- new net EOC2: IC4.10, JP1.37
- new net EOC3: IC7.10, JP2.33
- new net EOC4: IC8.10, JP2.27
- new net N$2: IC3.8, R5.1, TP8.1
- new net N$22: C11.2, IC8.4, R8.2
- new net N$3: C8.2, IC7.4, R6.2
- new net N$6: IC5.8, R7.1, TP9.1
- new net SCLK1: IC6.15, JP1.27
- new net SCLK2: IC4.15, JP1.33
- new net SCLK3: IC7.15, JP2.37
- new net SCLK4: IC8.15, JP2.31
- new net SDI1: IC6.12, JP1.29
- new net SDI2: IC4.12, JP1.35
- new net SDI3: IC7.12, JP2.35
- new net SDI4: IC8.12, JP2.29
- new net SDO1: IC6.13, JP1.28
- new net SDO2: IC4.13, JP1.34
- new net SDO3: IC7.13, JP2.38
- new net SDO4: IC8.13, JP2.32
- net !CS_PGA: now also JP2.12
- net +3V3: no longer C2.1, C3.1, C4.1, IC4.21, IC4.60, IC4.9
- net DIN_PGA: now also JP2.8
- net GND: now also C23.2, C24.2, IC10.2, IC4.14, IC4.5, IC4.6, IC6.14, IC6.5, IC6.6, IC7.14, IC7.5, IC7.6, IC8.14, IC8.5, IC8.6, IC9.2, R2.2, R4.1, R6.1, R8.1, TP1.1; no longer C11.2, C2.2, C5.2, C8.2, IC4.22, IC4.23, IC4.25, IC4.28, IC4.30, IC4.31, IC4.32, IC4.34, IC4.36, IC4.38, IC4.43, IC4.45, IC4.47, IC4.49, IC4.50, IC4.51, IC4.53, IC4.56, IC4.58, IC4.59, IC4.65, IC4.8, JP2.49
- net N$1: now also TP2.1
- net N$10: now also C5.1, IC4.3, R3.2; no longer IC3.8, R3.1
- net N$12: now also C2.1, IC6.3; no longer IC4.37
- net N$13: now also C5.2, IC4.4, R4.2; no longer IC4.39, R2.2
- net N$14: now also C2.2, IC6.4, R2.1; no longer IC4.42, R3.2
- net N$15: now also C8.1, IC7.3, R5.2; no longer IC4.44, R4.2
- net N$16: now also TP5.1
- net N$19: now also C11.1, IC8.3, R7.2; no longer C5.1, C6.1, C7.1, C8.1, IC4.26, IC4.27, IC4.33, IC4.40, IC4.48, IC4.54, IC4.55
- net N$4: now also TP3.1
- net N$5: now also TP4.1
- net N$8: now also TP6.1
- net N$9: now also R3.1, TP7.1; no longer R2.1
- net SCLK_PGA: now also JP2.10
- net VCC: now also C14.1, C24.1, IC10.1, IC10.3, IC9.1, IC9.3
Routing:
- net +3V3A: track 0.00 -> 115.3 mm
- net GND: track 1.17 -> 74.6 mm, vias 0 -> 31
- net +3V3D: track 0.00 -> 47.3 mm
- net SCLK_PGA: track 0.00 -> 46.6 mm
- net DIN_PGA: track 0.00 -> 46.6 mm
- net !CS_PGA: track 0.00 -> 46.4 mm
- net VCC: track 0.00 -> 37.3 mm, vias 0 -> 2
- net !CONVST2: track 0.00 -> 33.9 mm
- net !CS2: track 0.00 -> 31.4 mm
- net EOC2: track 0.00 -> 29.6 mm
- net SCLK3: track 0.00 -> 29.0 mm
- net SDO2: track 0.00 -> 28.9 mm
- net SDI2: track 0.00 -> 27.1 mm
- net SDI3: track 0.00 -> 26.2 mm
- net SDO3: track 0.00 -> 24.4 mm
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Other:
- board size 68.2 x 55.9 mm -> 55.9 x 55.9 mm

Commit message: rev 5.7.14 complete, sent for production
Parts:
- IC4: value ADS8327 -> MAX9939; device custom:TSSOP16 -> custom:UMAX10
- IC5: value MAX9939 -> ADS8327; device custom:UMAX10 -> custom:TSSOP16
- moved TP6 114.7 mm to (21.7, 42.5)
- moved TP7 110.9 mm to (21.7, 33.7)
- moved TP8 107.0 mm to (21.7, 24.8)
- moved TP9 103.1 mm to (21.7, 15.9)
- moved TP1 93.4 mm to (3.81, 47.9)
- moved TP2 88.9 mm to (12.3, 37.7)
- moved TP3 85.0 mm to (12.3, 28.8)
- moved TP4 81.1 mm to (12.3, 19.9)
- moved TP5 77.2 mm to (12.3, 11.0)
- moved IC5 29.4 mm to (30.9, 39.1)
- moved IC4 22.1 mm to (16.1, 13.7)
- moved IC6 8.89 mm to (30.9, 30.2)
Connections:
- net !CONVST1: now also IC5.9; no longer IC6.9
- net !CONVST2: now also IC6.9; no longer IC4.9
- net !CS1: now also IC5.11; no longer IC6.11
- net !CS2: now also IC6.11; no longer IC4.11
- net !CS_PGA: now also IC4.10; no longer IC5.10
- net +3V3A: now also IC4.9, IC5.1, IC5.7; no longer IC4.1, IC4.7, IC5.9
- net +3V3D: now also IC5.16; no longer IC4.16
- net DIN_PGA: now also IC4.2; no longer IC5.2
- net EOC1: now also IC5.10; no longer IC6.10
- net EOC2: now also IC6.10; no longer IC4.10
- net GND: now also IC4.3, IC4.4, IC5.14, IC5.5, IC5.6; no longer IC4.14, IC4.5, IC4.6, IC5.3, IC5.4
- net N$10: now also IC6.3; no longer IC4.3
- net N$12: now also IC5.3; no longer IC6.3
- net N$13: now also IC6.4; no longer IC4.4
- net N$14: now also IC5.4; no longer IC6.4
- net N$16: now also IC4.5; no longer IC5.5
- net N$6: now also IC4.8; no longer IC5.8
- net SCLK1: now also IC5.15; no longer IC6.15
- net SCLK2: now also IC6.15; no longer IC4.15
- net SCLK_PGA: now also IC4.1; no longer IC5.1
- net SDI1: now also IC5.12; no longer IC6.12
- net SDI2: now also IC6.12; no longer IC4.12
- net SDO1: now also IC5.13; no longer IC6.13
- net SDO2: now also IC6.13; no longer IC4.13
Routing:
- net N$9: track 4.25 -> 6.57 mm
- net N$6: track 4.25 -> 6.57 mm
- net N$8: track 4.25 -> 6.57 mm
- net N$2: track 4.25 -> 6.57 mm
- net N$1: track 8.42 -> 10.2 mm
- net N$5: track 8.42 -> 10.2 mm
- net N$16: track 8.42 -> 10.2 mm
- net N$4: track 8.42 -> 10.2 mm
Other:
- board text added: "AUVUA"
- board text added: "mojo afe"
- board text added: "r5.7.14"

Commit message: Widened board to properly fit Mojo. Rev 5.17.14 sent for prodution.
Parts:
- moved JP1 5.08 mm to (27.9, 57.1)
- moved C17 2.54 mm to (16.4, 37.1)
- moved C20 2.54 mm to (16.4, 29.6)
- moved C5 2.54 mm to (25.9, 33.0)
- moved IC2 2.54 mm to (16.1, 34.0)
- moved IC7 2.54 mm to (30.9, 23.9)
- moved R3 2.54 mm to (23.4, 34.0)
- moved C11 2.54 mm to (25.9, 15.2)
- moved IC4 2.54 mm to (16.1, 16.3)
- moved IC8 2.54 mm to (30.9, 15.0)
- moved R7 2.54 mm to (23.4, 16.3)
- moved R8 2.54 mm to (23.4, 14.2)
- moved TP5 2.54 mm to (12.3, 13.6)
- moved C1 2.54 mm to (28.8, 45.5)
- moved C10 2.54 mm to (28.8, 18.8)
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Routing:
- net SDI2: track 27.1 -> 29.7 mm
- net EOC1: track 17.6 -> 20.1 mm
- net !CONVST2: track 33.9 -> 36.4 mm
- net SCLK1: track 12.3 -> 14.9 mm
- net SDI3: track 26.2 -> 28.7 mm
- net SDI1: track 15.1 -> 17.6 mm
- net SCLK2: track 24.4 -> 26.9 mm
- net !CS2: track 31.4 -> 34.0 mm
- net !CONVST4: track 7.29 -> 9.83 mm
- net EOC4: track 11.6 -> 14.1 mm
- net SDO4: track 12.3 -> 14.8 mm
- net SDO2: track 28.9 -> 31.5 mm
- net SDO1: track 16.9 -> 19.4 mm
- net SCLK_PGA: track 46.6 -> 49.2 mm
- net SCLK4: track 16.8 -> 19.4 mm
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Other:
- board size 55.9 x 55.9 mm -> 55.9 x 61 mm
- board text added: "r5.17.14"
- board text removed: "r5.7.14"
