File: eagle/powermgr/powermgr.sch (EAGLE design)
At the start: 36 parts, among them IC1 PIC16F1455TSSOP-14, IC2 4027D, IC3 MCP1804, IC4 ACS756, Q1 BSS123, Q2 BSS123, X1 10104111-0001LF

Commit message: Added schmitt trigger to switch inputs. Sent rev 6.16.14 for production.
Parts:
- added IC5: 74HC2G14, custom:74HC2G14
- D1: value (none) -> PWR
- D2: value (none) -> MOTOR
- renumbered MOTOR to D2, PWR to D1
Connections:
- removed net N$2: C2.1, IC2B.CLK, JP2.1, R2.1
- new net N$15: C2.1, IC5.2A, JP2.1, R2.1
- new net N$17: IC2A.CLK, IC5.1Y
- new net N$18: IC2B.CLK, IC5.2Y
- net +5V: now also IC5.VCC
- net GND: now also IC5.GND
- net N$1: now also IC5.1A; no longer IC2A.CLK
Other:
- moved on the sheet: C1, C2, JP1, JP2, R1, R2
