File: eagle/peripheral/peripheral.sch (EAGLE design)
At the start: 0 parts

Commit message: Completed peripheral design layout.
Parts:
- added C1: 10u, resistor:C-EUC0805K
- added C2: 220n, resistor:C-EUC0603
- added C3: 100n, resistor:C-EUC0603
- added JP1: (no value), pinhead:PINHD-1X10
- added JP10, JP11, JP5, JP6, JP7, JP8, JP9: (no value), pinhead:PINHD-1X2
- added JP12: (no value), pinhead:PINHD-1X3
- added JP2, JP3: (no value), pinhead:PINHD-1X8
- added JP4: (no value), pinhead:PINHD-1X6
- added Q1, Q2: DMN4031SSD, peripheral:DMN4031SSD
- added Q3: BSS123, peripheral:BSS123
- added R1: 100k, resistor:R-US_R0805
- added R2, R3: 4.7k, resistor:R-US_R0603
- added U1: CHIPCAP2, peripheral:CHIPCAP2
- added X1, X2: (no value), con-wago-500:W237-103
Connections:
- new net +24V: X1-1.KL
- new net 0/RX1: JP2.8
- new net 1/TX1: JP2.7
- new net 10: JP1.8, Q2G$1.G
- new net 11: JP1.7, Q1G$2.G
- new net 12: JP1.6, U1.READY
- new net 13: JP1.5, Q1G$1.G
- new net 2: JP10.1, JP2.6, JP6.1, JP7.1, JP8.1, JP9.1
- new net 3: C1.1, JP2.5, JP5.1, R1.1
- new net 3.3V: JP3.4
- new net 4: JP2.4
- new net 5: JP2.3
- new net 5V: C2.1, C3.1, JP12.1, JP3.5, R1.2, R2.2, R3.2, U1.VDD
- new net 6: JP2.2
- new net 7: JP2.1
- new net 8: JP1.10, Q3.G
- new net 9: JP1.9, Q2G$2.G
- new net A0: JP4.1
- new net A1: JP4.2
- new net A2: JP4.3
- new net A3: JP4.4
- new net A4: JP4.5
- new net A5: JP12.2, JP4.6
- new net AREF: JP1.3
- new net BLUE_LED: Q2G$2.D, X2-3.KL
- new net GND: C1.2, C2.2, JP1.4, JP10.2, JP11.2, JP12.3, JP3.6, JP3.7, JP5.2, JP6.2, JP7.2, JP8.2, JP9.2, Q3.S, U1.GND
- new net GREEN_LED: Q2G$1.D, X2-2.KL
- new net IOREF: JP3.2
- new net N$2: JP11.1, Q3.D
- new net N$3: C3.2, U1.VCORE
- new net N$6: Q1G$1.S, Q1G$2.S, Q2G$1.S, Q2G$2.S, X1-2.KL
- new net RED_LED: Q1G$2.D, X2-1.KL
- new net RESET: JP3.3
- new net SCL: JP1.1, R2.1, U1.SCL
- new net SDA: JP1.2, R3.1, U1.SDA
- new net VIN: JP3.8
- new net WHITE_LED: Q1G$1.D, X1-3.KL
Other:
- note added: "Depth"
- note added: "GoPro Power"
- note added: "LED Indicators"
- note added: "Mission"
- note added: "Motor 1"
- note added: "Motor 2"
- note added: "Motor 3"
- note added: "Motor 4"
- note added: "Motor 5"
